File: front/led_pcb_l/led_pcb_l.sch (KiCad schematic (older format))
At the start: 4 parts

Commit message: adjust left pcb
Parts:
- renumbered D2 to D1, D4 to D3
Connections:
- net at D1.1 (K), D3.2 (A): now also R1.1; no longer B1.1
- net at D1.2 (A), D3.1 (K): now also B1.1; no longer R1.1
Other:
- moved on the sheet: D1
Changed lines of the file:
@@
 $EndDescr
 $Comp
-L Device:LED D2
+L Device:LED D1
 U 1 1 5E2AF667
 P 2700 1500
-F 0 "D2" H 2693 1716 50  0000 C CNN
+F 0 "D1" H 2693 1716 50  0000 C CNN
 F 1 "LED" H 2693 1625 50  0000 C CNN
 F 2 "LED_SMD:LED_1206_3216Metric" H 2700 1500 50  0001 C CNN
 F 3 "~" H 2700 1500 50  0001 C CNN
 	1    2700 1500
-	0    1    1    0
+	0    -1   -1   0
 $EndComp
 $Comp
-L Device:D D4
+L Device:D D3
 U 1 1 5E2AFDF7
 P 1900 1500
-F 0 "D4" H 1900 1716 50  0000 C CNN
+F 0 "D3" H 1900 1716 50  0000 C CNN
 F 1 "D" H 1900 1625 50  0000 C CNN
 F 2 "Diode_SMD:D_0603_1608Metric" H 1900 1500 50  0001 C CNN
 F 3 "~" H 1900 1500 50  0001 C CNN
 	1    1900 1500
-	0    -1   -1   0
+	0    1    1    0
 $EndComp
 $Comp
@@
 $EndComp
 Wire Wire Line
-	2700 1350 1900 1350
+	1300 1350 1900 1350
 Wire Wire Line
-	1900 1350 1300 1350
+	1300 1650 1900 1650
 Connection ~ 1900 1350
 Wire Wire Line
-	1300 1650 1900 1650
+	1900 1350 2700 1350
+Connection ~ 1900 1650
 Wire Wire Line
-	2700 1650 1900 1650
-Connection ~ 1900 1650
+	1900 1650 2700 1650
 $EndSCHEMATC
