File: front/led_pcb_r/led_pcb_r.kicad_pcb (KiCad board)
At the start: 2 copper layers, 6 x 29.3 mm, 6 parts

Commit message: adjust right pcb
Other:
- outline, holes or cut-outs redrawn
- board text added: "A"
- board text added: "B"
- board text added: "CG"
- board text added: "Side"
